Commit message: diminuindo o peso do robo

File: robot_description/urdf/robot_parts/carcaca.xacro (robot description, xacro)
@@ -12,5 +12,5 @@
         <link name="${base_link}">
             <inertial>
-                <mass value="2.4" />
+                <mass value="1.9" />
                 <origin rpy="0  0  3.14" xyz="0  0  0.0118" />
                 <inertia ixx="0.019995" ixy="0.0" ixz="0.0"

File: robot_description/urdf/robot_parts/piston.xacro (robot description, xacro)
@@ -20,5 +20,5 @@
         <link name="${prefix}">
             <inertial>
-                <mass value="0.3" />
+                <mass value="0.2" />
                 <origin rpy="0  0  0" xyz="0 0 0" />
                 <inertia ixx="0" ixy="0" ixz="0" iyy="0" iyz="0" izz="0" />

File: robot_description/urdf/robot_parts/traction_wheel.xacro (robot description, xacro)
@@ -21,5 +21,5 @@
         <link name="${prefix}">
             <inertial>
-                <mass value="1" />
+                <mass value="0.7" />
                 <origin rpy="0 0 0" xyz="0 0 0" />
                 <inertia ixx="0.001" ixy="0.0" ixz="0.0"

File: robot_description/urdf/robot_parts/tray.xacro (robot description, xacro)
@@ -19,5 +19,5 @@
         <link name="${prefix}">
             <inertial>
-                <mass value="0.5" />
+                <mass value="0.2" />
                 <origin rpy="0 0 0" xyz="0 0 0" />
                 <inertia ixx="0" ixy="0.0" ixz="0.0" iyy="0" iyz="0.0" izz="0" />
